File: hardware/power_supply.kicad_sch (KiCad schematic)
At the start: 20 parts, among them Q1 IRF740, U2 AP63203WU, U5 MAX1771xSA

Commit message: Update.
Parts:
- renumbered C12 to C1, C14 to C2, C8 to C4, C4 to C5, C5 to C6, C13 to C7, C11 to C8, D4 to D3, L2 to L1, L1 to L2, R18 to R1, R19 to R2, R20 to R3, U2 to U1, U5 to U2
Changed lines of the file:
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@@
 		(dnp no)
 		(fields_autoplaced yes)
-		(property "Reference" "L2"
+		(property "Reference" "L1"
 			(at 109.22 81.28 90)
 			(effects
@@
 			(project ""
 				(path "/90430e5f-7049-4de8-b92d-f897c4a89819/3e544bdc-8ef6-4ae7-86a5-8f5d44c9c569"
-					(reference "L2")
+					(reference "L1")
 					(unit 1)
 				)
@@
 		(dnp no)
 		(fields_autoplaced yes)
-		(property "Reference" "R18"
+		(property "Reference" "R1"
 			(at 127 118.1099 0)
 			(effects
@@
 			(project ""
 				(path "/90430e5f-7049-4de8-b92d-f897c4a89819/3e544bdc-8ef6-4ae7-86a5-8f5d44c9c569"
-					(reference "R18")
+					(reference "R1")
 					(unit 1)
 				)
@@
 		(dnp no)
 		(fields_autoplaced yes)
-		(property "Reference" "U2"
+		(property "Reference" "U1"
 			(at 86.36 44.45 0)
 			(effects
@@
 			(project "qw"
 				(path "/90430e5f-7049-4de8-b92d-f897c4a89819/3e544bdc-8ef6-4ae7-86a5-8f5d44c9c569"
-					(reference "U2")
+					(reference "U1")
 					(unit 1)
 				)
@@
 		(on_board yes)
 		(dnp no)
-		(property "Reference" "L1"
+		(property "Reference" "L2"
 			(at 109.2199 53.34 0)
 			(effects
@@
 			(project "qw"
 				(path "/90430e5f-7049-4de8-b92d-f897c4a89819/3e544bdc-8ef6-4ae7-86a5-8f5d44c9c569"
-					(reference "L1")
+					(reference "L2")
 					(unit 1)
 				)
@@
 		(on_board yes)
 		(dnp no)
-		(property "Reference" "C5"
+		(property "Reference" "C6"
 			(at 125.73 59.6899 0)
 			(effects
@@
 			(project "qw"
 				(path "/90430e5f-7049-4de8-b92d-f897c4a89819/3e544bdc-8ef6-4ae7-86a5-8f5d44c9c569"
-					(reference "C5")
+					(reference "C6")
 					(unit 1)
 				)
@@
 		(dnp no)
 		(fields_autoplaced yes)
-		(property "Reference" "C14"
+		(property "Reference" "C2"
 			(at 57.15 116.8399 0)
 			(effects
@@
 			(project "qw"
 				(path "/90430e5f-7049-4de8-b92d-f897c4a89819/3e544bdc-8ef6-4ae7-86a5-8f5d44c9c569"
-					(reference "C14")
+					(reference "C2")
 					(unit 1)
 				)
@@
 		(dnp no)
 		(fields_autoplaced yes)
-		(property "Reference" "U5"
+		(property "Reference" "U2"
 			(at 89.7733 93.98 0)
 			(effects
@@
 			(project ""
 				(path "/90430e5f-7049-4de8-b92d-f897c4a89819/3e544bdc-8ef6-4ae7-86a5-8f5d44c9c569"
-					(reference "U5")
+					(reference "U2")
 					(unit 1)
 				)
@@
 		(on_board yes)
 		(dnp no)
-		(property "Reference" "C4"
+		(property "Reference" "C5"
 			(at 106.68 46.9899 0)
 			(effects
@@
 			(project "qw"
 				(path "/90430e5f-7049-4de8-b92d-f897c4a89819/3e544bdc-8ef6-4ae7-86a5-8f5d44c9c569"
-					(reference "C4")
+					(reference "C5")
 					(unit 1)
 				)
@@
 		(dnp no)
 		(fields_autoplaced yes)
-		(property "Reference" "C11"
+		(property "Reference" "C8"
 			(at 180.34 121.9199 0)
 			(effects
@@
 			(project ""
 				(path "/90430e5f-7049-4de8-b92d-f897c4a89819/3e544bdc-8ef6-4ae7-86a5-8f5d44c9c569"
-					(reference "C11")
+					(reference "C8")
 					(unit 1)
 				)
@@
 		(dnp no)
 		(fields_autoplaced yes)
-		(property "Reference" "C13"
+		(property "Reference" "C7"
 			(at 147.32 121.0309 0)
 			(effects
@@
 			(project ""
 				(path "/90430e5f-7049-4de8-b92d-f897c4a89819/3e544bdc-8ef6-4ae7-86a5-8f5d44c9c569"
-					(reference "C13")
+					(reference "C7")
 					(unit 1)
 				)
@@
 		(dnp no)
 		(fields_autoplaced yes)
-		(property "Reference" "C8"
+		(property "Reference" "C4"
 			(at 77.47 118.1099 0)
 			(effects
@@
 			(project ""
 				(path "/90430e5f-7049-4de8-b92d-f897c4a89819/3e544bdc-8ef6-4ae7-86a5-8f5d44c9c569"
-					(reference "C8")
+					(reference "C4")
 					(unit 1)
 				)
@@
 		(dnp no)
 		(fields_autoplaced yes)
-		(property "Reference" "D4"
+		(property "Reference" "D3"
 			(at 139.7 80.01 0)
 			(effects
@@
 			(project ""
 				(path "/90430e5f-7049-4de8-b92d-f897c4a89819/3e544bdc-8ef6-4ae7-86a5-8f5d44c9c569"
-					(reference "D4")
+					(reference "D3")
 					(unit 1)
 				)
@@
 		(dnp no)
 		(fields_autoplaced yes)
-		(property "Reference" "R20"
+		(property "Reference" "R3"
 			(at 161.29 121.9199 0)
 			(effects
@@
 			(project "qw"
 				(path "/90430e5f-7049-4de8-b92d-f897c4a89819/3e544bdc-8ef6-4ae7-86a5-8f5d44c9c569"
-					(reference "R20")
+					(reference "R3")
 					(unit 1)
 				)
@@
 		(dnp no)
 		(fields_autoplaced yes)
-		(property "Reference" "C12"
+		(property "Reference" "C1"
 			(at 39.37 115.9509 0)
 			(effects
@@
 			(project ""
 				(path "/90430e5f-7049-4de8-b92d-f897c4a89819/3e544bdc-8ef6-4ae7-86a5-8f5d44c9c569"
-					(reference "C12")
+					(reference "C1")
 					(unit 1)
 				)
@@
 		(dnp no)
 		(fields_autoplaced yes)
-		(property "Reference" "R19"
+		(property "Reference" "R2"
 			(at 161.29 92.7099 0)
 			(effects
@@
 			(project "qw"
 				(path "/90430e5f-7049-4de8-b92d-f897c4a89819/3e544bdc-8ef6-4ae7-86a5-8f5d44c9c569"
-					(reference "R19")
-					(unit 1)
-				)
+					(reference "R2")
+					(unit 1)
+				)

Commit message: Add HT psu.
Parts:
- C1: value C_Polarized -> 100uF; footprint (none) -> Capacitor_Tantalum_SMD:CP_EIA-3528-15_AVX-H_HandSolder
- C2, C4: value C -> 100nF; footprint (none) -> Capacitor_SMD:C_0805_2012Metric
- C7: value C_Polarized -> 4.7uF; footprint (none) -> Capacitor_SMD:C_0805_2012Metric
- C8: value C -> 100nF; footprint (none) -> Capacitor_SMD:C_1210_3225Metric_Pad1.33x2.70mm_HandSolder
- D3: footprint (none) -> Capacitor_SMD:C_1210_3225Metric_Pad1.33x2.70mm_HandSolder
- L1: value L -> 100uH; footprint (none) -> Inductor_SMD:L_APV_APH1050
- Q1: footprint Package_TO_SOT_THT:TO-220-3_Vertical -> Package_TO_SOT_SMD:TO-263-2
- R1: value R -> 0.05; footprint (none) -> Resistor_SMD:R_1206_3216Metric
- R2: value R -> 1.5M; footprint (none) -> Resistor_SMD:R_1206_3216Metric
- R3: value R -> 10k; footprint (none) -> Resistor_SMD:R_1206_3216Metric
- RV1: footprint (none) -> Potentiometer_SMD:Potentiometer_Bourns_3314G_Vertical
Connections:
- net at U2.3 (FB): now also R2.2, RV1.3
Changed lines of the file:
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@@
+	)
+	(junction
+		(at 158.75 100.33)
+		(diameter 0)
+		(color 0 0 0 0)
 	)
 	(junction
@@
 	(wire
 		(pts
-			(xy 158.75 97.79) (xy 158.75 102.87)
+			(xy 158.75 97.79) (xy 158.75 100.33)
 		)
 		(stroke
@@
 	(wire
 		(pts
+			(xy 97.79 109.22) (xy 151.13 109.22)
+		)
+		(stroke
+			(width 0)
+			(type default)
+		)
+	)
+	(wire
+		(pts
 			(xy 124.46 123.19) (xy 124.46 139.7)
 		)
@@
 	(wire
 		(pts
+			(xy 151.13 100.33) (xy 158.75 100.33)
+		)
+		(stroke
+			(width 0)
+			(type default)
+		)
+	)
+	(wire
+		(pts
 			(xy 176.53 86.36) (xy 184.15 86.36)
 		)
@@
 	(wire
 		(pts
+			(xy 151.13 109.22) (xy 151.13 100.33)
+		)
+		(stroke
+			(width 0)
+			(type default)
+		)
+	)
+	(wire
+		(pts
 			(xy 96.52 57.15) (xy 118.11 57.15)
 		)
@@
 		(pts
 			(xy 35.56 121.92) (xy 35.56 139.7)
+		)
+		(stroke
+			(width 0)
+			(type default)
+		)
+	)
+	(wire
+		(pts
+			(xy 158.75 100.33) (xy 158.75 102.87)
 		)
 		(stroke
@@
 			)
 		)
-		(property "Value" "L"
+		(property "Value" "100uH"
 			(at 109.22 83.82 90)
 			(effects
@@
 			)
 		)
-		(property "Footprint" ""
+		(property "Footprint" "Inductor_SMD:L_APV_APH1050"
 			(at 109.22 86.36 0)
 			(effects
@@
 			)
 		)
-		(property "Value" "R"
+		(property "Value" "0.05"
 			(at 127 120.6499 0)
 			(effects
@@
 			)
 		)
-		(property "Footprint" ""
+		(property "Footprint" "Resistor_SMD:R_1206_3216Metric"
 			(at 122.682 119.38 90)
 			(effects
@@
 			)
 		)
-		(property "Value" "C"
+		(property "Value" "100nF"
 			(at 57.15 119.3799 0)
 			(effects
@@
 			)
 		)
-		(property "Footprint" ""
+		(property "Footprint" "Capacitor_SMD:C_0805_2012Metric"
 			(at 54.3052 121.92 0)
 			(effects
@@
 			)
 		)
-		(property "Value" "C"
+		(property "Value" "100nF"
 			(at 180.34 124.4599 0)
 			(effects
@@
 			)
 		)
-		(property "Footprint" ""
+		(property "Footprint" "Capacitor_SMD:C_1210_3225Metric_Pad1.33x2.70mm_HandSolder"
 			(at 177.4952 127 0)
 			(effects
@@
 			)
 		)
-		(property "Value" "C_Polarized"
+		(property "Value" "4.7uF"
 			(at 147.32 123.5709 0)
 			(effects
@@
 			)
 		)
-		(property "Footprint" ""
+		(property "Footprint" "Capacitor_SMD:C_0805_2012Metric"
 			(at 144.4752 127 0)
 			(effects
@@
 			)
 		)
-		(property "Value" "C"
+		(property "Value" "100nF"
 			(at 77.47 120.6499 0)
 			(effects
@@
 			)
 		)
-		(property "Footprint" ""
+		(property "Footprint" "Capacitor_SMD:C_0805_2012Metric"
 			(at 74.6252 123.19 0)
 			(effects
@@
 			)
 		)
-		(property "Footprint" ""
+		(property "Footprint" "Capacitor_SMD:C_1210_3225Metric_Pad1.33x2.70mm_HandSolder"
 			(at 139.7 86.36 0)
 			(effects
@@
 			)
 		)
-		(property "Value" "R"
+		(property "Value" "10k"
 			(at 161.29 124.4599 0)
 			(effects
@@
 			)
 		)
-		(property "Footprint" ""
+		(property "Footprint" "Resistor_SMD:R_1206_3216Metric"
 			(at 156.972 123.19 90)
 			(effects
@@
 			)
 		)
-		(property "Value" "C_Polarized"
+		(property "Value" "100uF"
 			(at 39.37 118.4909 0)
 			(effects
@@
 			)
 		)
-		(property "Footprint" ""
+		(property "Footprint" "Capacitor_Tantalum_SMD:CP_EIA-3528-15_AVX-H_HandSolder"
 			(at 36.5252 121.92 0)
 			(effects
@@
 			)
 		)
-		(property "Value" "R"
+		(property "Value" "1.5M"
 			(at 161.29 95.2499 0)
 			(effects
@@
 			)
 		)
-		(property "Footprint" ""
+		(property "Footprint" "Resistor_SMD:R_1206_3216Metric"
 			(at 156.972 93.98 90)
 			(effects
@@
 			)
 		)
-		(property "Footprint" "Package_TO_SOT_THT:TO-220-3_Vertical"
+		(property "Footprint" "Package_TO_SOT_SMD:TO-263-2"
 			(at 127 103.505 0)
 			(effects
@@
 			)
 		)
-		(property "Footprint" ""
+		(property "Footprint" "Potentiometer_SMD:Potentiometer_Bourns_3314G_Vertical"
 			(at 158.75 106.68 0)
 			(effects

Commit message: Rename nixie's names to have the right order.
Parts:
- Q1: footprint Package_TO_SOT_SMD:TO-263-2 -> Package_TO_SOT_THT:TO-220-3_Vertical
Changed lines of the file:
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@@
 			)
 		)
-		(property "Footprint" "Package_TO_SOT_SMD:TO-263-2"
+		(property "Footprint" "Package_TO_SOT_THT:TO-220-3_Vertical"
 			(at 127 103.505 0)
 			(effects

Commit message: Fix DRC errors.
Parts:
- Q1: footprint Package_TO_SOT_THT:TO-220-3_Vertical -> Package_TO_SOT_SMD:TO-263-2
Changed lines of the file:
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@@
 			)
 		)
-		(property "Footprint" "Package_TO_SOT_THT:TO-220-3_Vertical"
+		(property "Footprint" "Package_TO_SOT_SMD:TO-263-2"
 			(at 127 103.505 0)
 			(effects

Commit message: Remove POLarity setup, needs 12V to be not reversed.
Parts:
- R1: footprint Resistor_SMD:R_1206_3216Metric -> Resistor_SMD:R_0805_2012Metric
Changed lines of the file:
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@@
 			)
 		)
-		(property "Footprint" "Resistor_SMD:R_1206_3216Metric"
+		(property "Footprint" "Resistor_SMD:R_0805_2012Metric"
 			(at 122.682 119.38 90)
 			(effects

Commit message: Fix tube resistors and capacitors with 805.
Parts:
- Q1: footprint Package_TO_SOT_SMD:TO-263-2 -> Package_TO_SOT_THT:TO-220-3_Vertical
Changed lines of the file:
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@@
 			)
 		)
-		(property "Footprint" "Package_TO_SOT_SMD:TO-263-2"
+		(property "Footprint" "Package_TO_SOT_THT:TO-220-3_Vertical"
 			(at 127 103.505 0)
 			(effects

Commit message: Rework  3.3v power supply (fix error on fb loop). Put 1206 back on HV part.
Parts:
- added C16: 22uF, Capacitor_SMD:C_1206_3216Metric, symbol Device:C
- C2, C4, C8: value 100nF -> C
- C3: value 10uF 25V X7R -> 10uF; footprint Capacitor_SMD:C_0805_2012Metric -> Capacitor_SMD:C_1206_3216Metric
- C5: value 100µF / 10 V / X5R / 1210 -> 100nF; footprint Capacitor_SMD:C_1210_3225Metric -> Capacitor_SMD:C_0805_2012Metric
- C6: value 22uF 10V X7R -> 22uF; footprint Capacitor_SMD:C_0805_2012Metric -> Capacitor_SMD:C_1206_3216Metric
- L2: value 4.7uH 2A shielded -> 6.8uH
Connections:
- net 3.3V: now also C16.1
- net GND: now also C16.2
- net at C5.1, U1.5 (SW): now also L2.1
- net at C5.2, U1.6 (BST): no longer L2.1
Other:
- moved on the sheet: C3, C5, C6, D1, D2, L2, U1
