File: hardware/power_supply.kicad_sch (KiCad schematic)
At the start: 21 parts, among them Q1 IRF740, U1 AP63203WU, U2 MAX1771xSA

Commit message: Fix DRC errors.
Parts:
- Q1: footprint Package_TO_SOT_THT:TO-220-3_Vertical -> Package_TO_SOT_SMD:TO-263-2
Changed lines of the file:
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@@
 			)
 		)
-		(property "Footprint" "Package_TO_SOT_THT:TO-220-3_Vertical"
+		(property "Footprint" "Package_TO_SOT_SMD:TO-263-2"
 			(at 127 103.505 0)
 			(effects

Commit message: Fix most of ERC on schema. Add missing wire on RV1. Add PWR_FLG on GND to avoid error. Add resistor for unused SPI_OUT of HV5622. Add PTC on 3v3 supply.
Parts:
- added TH1: Thermistor_PTC, Resistor_SMD:R_1206_3216Metric, symbol Device:Thermistor_PTC
Connections:
- net at C3.1, U1.2 (EN), U1.3 (IN): now also TH1.1; no longer D1.1 (K), D2.1 (K)
- net at R3.1, RV1.1: now also RV1.2
- new net: D1.1 (K), D2.1 (K), TH1.2
Other:
- moved on the sheet: D1, D2

Commit message: Update PCB.
Parts:
- removed TH1: Thermistor_PTC, Resistor_SMD:R_1206_3216Metric, symbol Device:Thermistor_PTC
- C2, C4, C8: value C -> 100nF
- D3: value D -> ES2F
- R2, R3: footprint Resistor_SMD:R_1206_3216Metric -> Resistor_SMD:R_0805_2012Metric
- RV1: value R_Potentiometer_Trim -> 5K
Connections:
- net at C3.1, U1.2 (EN), U1.3 (IN): now also D1.1 (K), D2.1 (K)
Other:
- moved on the sheet: C3, D1, D2
Changed lines of the file:
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@@
-	)
-	(junction
-		(at 67.31 35.56)
-		(diameter 0)
-		(color 0 0 0 0)
 	)
 	(junction
@@
 	(wire
 		(pts
-			(xy 24.13 24.13) (xy 36.83 24.13)
+			(xy 25.4 40.64) (xy 38.1 40.64)
 		)
 		(stroke
@@
 	(wire
 		(pts
+			(xy 67.31 54.61) (xy 67.31 52.07)
+		)
+		(stroke
+			(width 0)
+			(type default)
+		)
+	)
+	(wire
+		(pts
 			(xy 111.76 52.07) (xy 111.76 44.45)
 		)
@@
 	(wire
 		(pts
-			(xy 67.31 24.13) (xy 67.31 35.56)
+			(xy 67.31 40.64) (xy 67.31 52.07)
 		)
 		(stroke
@@
 	(wire
 		(pts
-			(xy 44.45 24.13) (xy 67.31 24.13)
+			(xy 45.72 40.64) (xy 67.31 40.64)
 		)
 		(stroke
@@
 	(wire
 		(pts
-			(xy 67.31 35.56) (xy 67.31 40.64)
-		)
-		(stroke
-			(width 0)
-			(type default)
-		)
-	)
-	(wire
-		(pts
 			(xy 86.36 52.07) (xy 86.36 57.15)
 		)
@@
 	(wire
 		(pts
-			(xy 67.31 48.26) (xy 67.31 52.07)
-		)
-		(stroke
-			(width 0)
-			(type default)
-		)
-	)
-	(wire
-		(pts
 			(xy 158.75 127) (xy 158.75 139.7)
 		)
@@
 	(wire
 		(pts
-			(xy 24.13 35.56) (xy 36.83 35.56)
+			(xy 25.4 52.07) (xy 38.1 52.07)
 		)
 		(stroke
@@
 	(wire
 		(pts
-			(xy 44.45 35.56) (xy 67.31 35.56)
-		)
-		(stroke
-			(width 0)
-			(type default)
-		)
-	)
-	(wire
-		(pts
-			(xy 67.31 64.77) (xy 67.31 59.69)
+			(xy 45.72 52.07) (xy 67.31 52.07)
+		)
+		(stroke
+			(width 0)
+			(type default)
+		)
+	)
+	(wire
+		(pts
+			(xy 67.31 64.77) (xy 67.31 62.23)
 		)
 		(stroke
@@
 	(hierarchical_label "12V"
 		(shape input)
-		(at 24.13 24.13 180)
+		(at 25.4 40.64 180)
 		(effects
 			(font
@@
 	(hierarchical_label "5V"
 		(shape input)
-		(at 24.13 35.56 180)
+		(at 25.4 52.07 180)
 		(effects
 			(font
@@
 	(symbol
 		(lib_id "Device:C")
-		(at 67.31 55.88 0)
+		(at 67.31 58.42 0)
 		(unit 1)
 		(exclude_from_sim no)
@@
 		(dnp no)
 		(property "Reference" "C3"
-			(at 71.12 54.6099 0)
+			(at 71.12 57.1499 0)
 			(effects
 				(font
@@
 		)
 		(property "Value" "10uF"
-			(at 71.12 56.896 0)
+			(at 71.12 59.436 0)
 			(effects
 				(font
@@
 		)
 		(property "Footprint" "Capacitor_SMD:C_1206_3216Metric"
-			(at 68.2752 59.69 0)
+			(at 68.2752 62.23 0)
 			(effects
 				(font
@@
 		)
 		(property "Datasheet" "~"
-			(at 67.31 55.88 0)
+			(at 67.31 58.42 0)
 			(effects
 				(font
@@
 		)
 		(property "Description" "Unpolarized capacitor"
-			(at 67.31 55.88 0)
+			(at 67.31 58.42 0)
 			(effects
 				(font
@@
 	(symbol
 		(lib_id "Device:D_Schottky")
-		(at 40.64 35.56 180)
+		(at 41.91 52.07 180)
 		(unit 1)
 		(exclude_from_sim no)
@@
 		(dnp no)
 		(property "Reference" "D2"
-			(at 40.64 29.21 0)
+			(at 41.91 45.72 0)
 			(effects
 				(font
@@
 		)
 		(property "Value" "D_Schottky"
-			(at 40.64 31.75 0)
+			(at 41.91 48.26 0)
 			(effects
 				(font
@@
 		)
 		(property "Footprint" "Diode_SMD:D_2114_3652Metric_Pad1.85x3.75mm_HandSolder"
-			(at 40.64 35.56 0)
+			(at 41.91 52.07 0)
 			(effects
 				(font
@@
 		)
 		(property "Datasheet" "~"
-			(at 40.64 35.56 0)
+			(at 41.91 52.07 0)
 			(effects
 				(font
@@
 		)
 		(property "Description" "Schottky diode"
-			(at 40.64 35.56 0)
+			(at 41.91 52.07 0)
 			(effects
 				(font
@@
 	(symbol
 		(lib_id "Device:D_Schottky")
-		(at 40.64 24.13 180)
+		(at 41.91 40.64 180)
 		(unit 1)
 		(exclude_from_sim no)
@@
 		(fields_autoplaced yes)
 		(property "Reference" "D1"
-			(at 40.9575 17.78 0)
+			(at 42.2275 34.29 0)
 			(effects
 				(font
@@
 		)
 		(property "Value" "D_Schottky"
-			(at 40.9575 20.32 0)
+			(at 42.2275 36.83 0)
 			(effects
 				(font
@@
 		)
 		(property "Footprint" "Diode_SMD:D_2114_3652Metric_Pad1.85x3.75mm_HandSolder"
-			(at 40.64 24.13 0)
+			(at 41.91 40.64 0)
 			(effects
 				(font
@@
 		)
 		(property "Datasheet" "~"
-			(at 40.64 24.13 0)
+			(at 41.91 40.64 0)
 			(effects
 				(font
@@
 		)
 		(property "Description" "Schottky diode"
-			(at 40.64 24.13 0)
+			(at 41.91 40.64 0)
 			(effects
 				(font
@@
 			)
 		)
-		(property "Value" "C"
+		(property "Value" "100nF"
 			(at 57.15 119.3799 0)
 			(effects
@@
 			)
 		)
-		(property "Value" "C"
+		(property "Value" "100nF"
 			(at 180.34 124.4599 0)
 			(effects
@@
 			)
 		)
-		(property "Value" "C"
+		(property "Value" "100nF"
 			(at 77.47 120.6499 0)
 			(effects
@@
 			)
 		)
-		(property "Value" "D"
+		(property "Value" "ES2F"
 			(at 139.7 82.55 0)
 			(effects
@@
 			)
 		)
-		(property "Footprint" "Resistor_SMD:R_1206_3216Metric"
+		(property "Footprint" "Resistor_SMD:R_0805_2012Metric"
 			(at 156.972 123.19 90)
 			(effects
@@
 				(path "/90430e5f-7049-4de8-b92d-f897c4a89819/3e544bdc-8ef6-4ae7-86a5-8f5d44c9c569"
 					(reference "R3")
-					(unit 1)
-				)
-			)
-		)
-	)
-	(symbol
-		(lib_id "Device:Thermistor_PTC")
-		(at 67.31 44.45 180)
-		(unit 1)
-		(exclude_from_sim no)
-		(in_bom yes)
-		(on_board yes)
-		(dnp no)
-		(property "Reference" "TH1"
-			(at 61.214 42.672 0)
-			(effects
-				(font
-					(size 1.27 1.27)
-				)
-				(justify right)
-			)
-		)
-		(property "Value" "Thermistor_PTC"
-			(at 50.292 45.466 0)
-			(effects
-				(font
-					(size 1.27 1.27)
-				)
-				(justify right)
-			)
-		)
-		(property "Footprint" "Resistor_SMD:R_1206_3216Metric"
-			(at 66.04 39.37 0)
-			(effects
-				(font
-					(size 1.27 1.27)
-				)
-				(justify left)
-				(hide yes)
-			)
-		)
-		(property "Datasheet" "~"
-			(at 67.31 44.45 0)
-			(effects
-				(font
-					(size 1.27 1.27)
-				)
-				(hide yes)
-			)
-		)
-		(property "Description" "Temperature dependent resistor, positive temperature coefficient"
-			(at 67.31 44.45 0)
-			(effects
-				(font
-					(size 1.27 1.27)
-				)
-				(hide yes)
-			)
-		)
-		(pin "2"
-		)
-		(pin "1"
-		)
-		(instances
-			(project ""
-				(path "/90430e5f-7049-4de8-b92d-f897c4a89819/3e544bdc-8ef6-4ae7-86a5-8f5d44c9c569"
-					(reference "TH1")
 					(unit 1)
 				)
@@
 			)
 		)
-		(property "Footprint" "Resistor_SMD:R_1206_3216Metric"
+		(property "Footprint" "Resistor_SMD:R_0805_2012Metric"
 			(at 156.972 93.98 90)
 			(effects
@@
 			)
 		)
-		(property "Value" "R_Potentiometer_Trim"
+		(property "Value" "5K"
 			(at 161.29 107.9499 0)
 			(effects

Commit message: Rework HT PSU placement.
Parts:
- added TP2: TestPoint, TestPoint:TestPoint_Pad_D1.5mm, symbol Connector:TestPoint
Connections:
- net 3.3V: now also TP2.1
Changed lines of the file:
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@@
+	)
+	(junction
+		(at 162.56 57.15)
+		(diameter 0)
+		(color 0 0 0 0)
 	)
 	(junction
@@
 	(wire
 		(pts
-			(xy 149.86 57.15) (xy 171.45 57.15)
+			(xy 149.86 57.15) (xy 162.56 57.15)
 		)
 		(stroke
@@
 		(pts
 			(xy 67.31 64.77) (xy 67.31 62.23)
+		)
+		(stroke
+			(width 0)
+			(type default)
+		)
+	)
+	(wire
+		(pts
+			(xy 162.56 57.15) (xy 171.45 57.15)
 		)
 		(stroke
@@
 					(unit 1)
 				)
+			)
+		)
+	)
+	(symbol
+		(lib_id "Connector:TestPoint")
+		(at 162.56 57.15 0)
+		(unit 1)
+		(exclude_from_sim no)
+		(in_bom yes)
+		(on_board yes)
+		(dnp no)
+		(property "Reference" "TP2"
+			(at 158.242 49.022 0)
+			(effects
+				(font
+					(size 1.27 1.27)
+				)
+				(justify left)
+			)
+		)
+		(property "Value" "TestPoint"
+			(at 158.242 51.562 0)
+			(effects
+				(font
+					(size 1.27 1.27)
+				)
+				(justify left)
+			)
+		)
+		(property "Footprint" "TestPoint:TestPoint_Pad_D1.5mm"
+			(at 167.64 57.15 0)
+			(effects
+				(font
+					(size 1.27 1.27)
+				)
+				(hide yes)
+			)
+		)
+		(property "Datasheet" "~"
+			(at 167.64 57.15 0)
+			(effects
+				(font
+					(size 1.27 1.27)
+				)
+				(hide yes)
+			)
+		)
+		(property "Description" "test point"
+			(at 162.56 57.15 0)
+			(effects
+				(font
+					(size 1.27 1.27)
+				)
+				(hide yes)
+			)
+		)
+		(pin "1"
+		)
+		(instances
+			(project "nixie_clock"
+				(path "/90430e5f-7049-4de8-b92d-f897c4a89819/3e544bdc-8ef6-4ae7-86a5-8f5d44c9c569"
+					(reference "TP2")
+					(unit 1)
+				)

Commit message: Center USB-C connector on PCB. Add testpoints.
Parts:
- renumbered TP2 to 3V3
Changed lines of the file:
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@@
 		(on_board yes)
 		(dnp no)
-		(property "Reference" "TP2"
+		(property "Reference" "3V3"
 			(at 158.242 49.022 0)
 			(effects
@@
 			(project "nixie_clock"
 				(path "/90430e5f-7049-4de8-b92d-f897c4a89819/3e544bdc-8ef6-4ae7-86a5-8f5d44c9c569"
-					(reference "TP2")
+					(reference "3V3")
 					(unit 1)
 				)

Commit message: Update components to match BOM.
Parts:
- C1: footprint Capacitor_Tantalum_SMD:CP_EIA-3528-15_AVX-H_HandSolder -> Capacitor_Tantalum_SMD:CP_EIA-7343-31_Kemet-D_HandSolder
- C7: footprint Capacitor_SMD:C_0805_2012Metric -> Capacitor_SMD:C_Elec_8x10.2
- D3: footprint Capacitor_SMD:C_1210_3225Metric_Pad1.33x2.70mm_HandSolder -> Diode_SMD:D_SMB
- RV1: footprint Potentiometer_SMD:Potentiometer_Bourns_3314G_Vertical -> Potentiometer_SMD:Potentiometer_Bourns_3224G_Horizontal
Changed lines of the file:
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@@
 			)
 		)
-		(property "Footprint" "Capacitor_SMD:C_0805_2012Metric"
+		(property "Footprint" "Capacitor_SMD:C_Elec_8x10.2"
 			(at 144.4752 127 0)
 			(effects
@@
 			)
 		)
-		(property "Footprint" "Capacitor_SMD:C_1210_3225Metric_Pad1.33x2.70mm_HandSolder"
+		(property "Footprint" "Diode_SMD:D_SMB"
 			(at 139.7 86.36 0)
 			(effects
@@
 			)
 		)
-		(property "Footprint" "Capacitor_Tantalum_SMD:CP_EIA-3528-15_AVX-H_HandSolder"
+		(property "Footprint" "Capacitor_Tantalum_SMD:CP_EIA-7343-31_Kemet-D_HandSolder"
 			(at 36.5252 121.92 0)
 			(effects
@@
 			)
 		)
-		(property "Footprint" "Potentiometer_SMD:Potentiometer_Bourns_3314G_Vertical"
+		(property "Footprint" "Potentiometer_SMD:Potentiometer_Bourns_3224G_Horizontal"
 			(at 158.75 106.68 0)
 			(effects

Commit message: Limitate inrush current (decoupling capacitors after PTCs). Add decoupling capacitors for VUSB.
Parts:
- removed C2: 100nF, Capacitor_SMD:C_0805_2012Metric, symbol Device:C
- added R16: 0, Resistor_SMD:R_1206_3216Metric, symbol Device:R
- D1, D2: footprint Diode_SMD:D_2114_3652Metric_Pad1.85x3.75mm_HandSolder -> Diode_SMD:D_SMB
Connections:
- net 3.3V: now also R16.1; no longer C16.1, C6.1, L2.2, U1.1 (FB)
- new net: C16.1, C6.1, L2.2, R16.2, U1.1 (FB)
Other:
- moved on the sheet: 3V3
Changed lines of the file:
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@@
 	)
 	(junction
-		(at 162.56 57.15)
+		(at 167.64 57.15)
 		(diameter 0)
 		(color 0 0 0 0)
@@
 	)
 	(junction
-		(at 53.34 86.36)
-		(diameter 0)
-		(color 0 0 0 0)
-	)
-	(junction
 		(at 158.75 113.03)
 		(diameter 0)
@@
 	(wire
 		(pts
-			(xy 53.34 139.7) (xy 53.34 121.92)
-		)
-		(stroke
-			(width 0)
-			(type default)
-		)
-	)
-	(wire
-		(pts
-			(xy 53.34 86.36) (xy 87.63 86.36)
-		)
-		(stroke
-			(width 0)
-			(type default)
-		)
-	)
-	(wire
-		(pts
-			(xy 53.34 86.36) (xy 53.34 114.3)
-		)
-		(stroke
-			(width 0)
-			(type default)
-		)
-	)
-	(wire
-		(pts
 			(xy 158.75 97.79) (xy 158.75 100.33)
 		)
@@
 	(wire
 		(pts
+			(xy 167.64 57.15) (xy 171.45 57.15)
+		)
+		(stroke
+			(width 0)
+			(type default)
+		)
+	)
+	(wire
+		(pts
 			(xy 97.79 109.22) (xy 151.13 109.22)
 		)
@@
 	(wire
 		(pts
-			(xy 149.86 57.15) (xy 162.56 57.15)
+			(xy 149.86 57.15) (xy 154.94 57.15)
 		)
 		(stroke
@@
 	(wire
 		(pts
-			(xy 162.56 57.15) (xy 171.45 57.15)
-		)
-		(stroke
-			(width 0)
-			(type default)
-		)
-	)
-	(wire
-		(pts
 			(xy 158.75 110.49) (xy 158.75 113.03)
 		)
@@
 	(wire
 		(pts
-			(xy 35.56 86.36) (xy 53.34 86.36)
+			(xy 35.56 86.36) (xy 87.63 86.36)
 		)
 		(stroke
@@
 		)
 	)
-	(hierarchical_label "GND"
-		(shape input)
-		(at 53.34 139.7 270)
-		(effects
-			(font
-				(size 1.27 1.27)
-			)
-			(justify right)
+	(wire
+		(pts
+			(xy 162.56 57.15) (xy 167.64 57.15)
+		)
+		(stroke
+			(width 0)
+			(type default)
 		)
 	)
@@
 	(symbol
 		(lib_id "Connector:TestPoint")
-		(at 162.56 57.15 0)
+		(at 167.64 57.15 0)
 		(unit 1)
 		(exclude_from_sim no)
@@
 		(dnp no)
 		(property "Reference" "3V3"
-			(at 158.242 49.022 0)
+			(at 163.322 49.022 0)
 			(effects
 				(font
@@
 		)
 		(property "Value" "TestPoint"
-			(at 158.242 51.562 0)
+			(at 163.322 51.562 0)
 			(effects
 				(font
@@
 		)
 		(property "Footprint" "TestPoint:TestPoint_Pad_D1.5mm"
+			(at 172.72 57.15 0)
+			(effects
+				(font
+					(size 1.27 1.27)
+				)
+				(hide yes)
+			)
+		)
+		(property "Datasheet" "~"
+			(at 172.72 57.15 0)
+			(effects
+				(font
+					(size 1.27 1.27)
+				)
+				(hide yes)
+			)
+		)
+		(property "Description" "test point"
 			(at 167.64 57.15 0)
-			(effects
-				(font
-					(size 1.27 1.27)
-				)
-				(hide yes)
-			)
-		)
-		(property "Datasheet" "~"
-			(at 167.64 57.15 0)
-			(effects
-				(font
-					(size 1.27 1.27)
-				)
-				(hide yes)
-			)
-		)
-		(property "Description" "test point"
-			(at 162.56 57.15 0)
 			(effects
 				(font
@@
 			)
 		)
-		(property "Footprint" "Diode_SMD:D_2114_3652Metric_Pad1.85x3.75mm_HandSolder"
+		(property "Footprint" "Diode_SMD:D_SMB"
 			(at 41.91 52.07 0)
 			(effects
@@
 			)
 		)
-		(property "Footprint" "Diode_SMD:D_2114_3652Metric_Pad1.85x3.75mm_HandSolder"
+		(property "Footprint" "Diode_SMD:D_SMB"
 			(at 41.91 40.64 0)
 			(effects
@@
 				(path "/90430e5f-7049-4de8-b92d-f897c4a89819/3e544bdc-8ef6-4ae7-86a5-8f5d44c9c569"
 					(reference "D1")
-					(unit 1)
-				)
-			)
-		)
-	)
-	(symbol
-		(lib_id "Device:C")
-		(at 53.34 118.11 0)
-		(unit 1)
-		(exclude_from_sim no)
-		(in_bom yes)
-		(on_board yes)
-		(dnp no)
-		(fields_autoplaced yes)
-		(property "Reference" "C2"
-			(at 57.15 116.8399 0)
-			(effects
-				(font
-					(size 1.27 1.27)
-				)
-				(justify left)
-			)
-		)
-		(property "Value" "100nF"
-			(at 57.15 119.3799 0)
-			(effects
-				(font
-					(size 1.27 1.27)
-				)
-				(justify left)
-			)
-		)
-		(property "Footprint" "Capacitor_SMD:C_0805_2012Metric"
-			(at 54.3052 121.92 0)
-			(effects
-				(font
-					(size 1.27 1.27)
-				)
-				(hide yes)
-			)
-		)
-		(property "Datasheet" "~"
-			(at 53.34 118.11 0)
-			(effects
-				(font
-					(size 1.27 1.27)
-				)
-				(hide yes)
-			)
-		)
-		(property "Description" "Unpolarized capacitor"
-			(at 53.34 118.11 0)
-			(effects
-				(font
-					(size 1.27 1.27)
-				)
-				(hide yes)
-			)
-		)
-		(pin "1"
-		)
-		(pin "2"
-		)
-		(instances
-			(project "qw"
-				(path "/90430e5f-7049-4de8-b92d-f897c4a89819/3e544bdc-8ef6-4ae7-86a5-8f5d44c9c569"
-					(reference "C2")
 					(unit 1)
 				)
@@
 					(unit 1)
 				)
+			)
+		)
+	)
+	(symbol
+		(lib_id "Device:R")
+		(at 158.75 57.15 270)
+		(unit 1)
+		(exclude_from_sim no)
+		(in_bom yes)
+		(on_board yes)
+		(dnp no)
+		(property "Reference" "R16"
+			(at 158.75 51.816 90)
+			(effects
+				(font
+					(size 1.27 1.27)
+				)
+			)
+		)
+		(property "Value" "0"
+			(at 158.75 54.356 90)
+			(effects
+				(font
+					(size 1.27 1.27)
+				)
+			)
+		)
+		(property "Footprint" "Resistor_SMD:R_1206_3216Metric"
+			(at 158.75 55.372 90)
+			(effects
+				(font
+					(size 1.27 1.27)
+				)
+				(hide yes)
+			)
+		)
+		(property "Datasheet" "~"
+			(at 158.75 57.15 0)
+			(effects
+				(font
+					(size 1.27 1.27)
+				)
+				(hide yes)
+			)
+		)
+		(property "Description" "Resistor"
+			(at 158.75 57.15 0)
+			(effects
+				(font
+					(size 1.27 1.27)
+				)
+				(hide yes)
+			)
+		)
+		(pin "1"
+		)
+		(pin "2"
+		)
+		(instances
+			(project "nixie_clock"
+				(path "/90430e5f-7049-4de8-b92d-f897c4a89819/3e544bdc-8ef6-4ae7-86a5-8f5d44c9c569"
+					(reference "R16")
+					(unit 1)
+				)

Commit message: Update, DRC ok.
Parts:
- added C2: 100nF, Capacitor_SMD:C_0805_2012Metric, symbol Device:C
- L2: footprint Inductor_SMD:L_1210_3225Metric -> Inductor_SMD:L_Bourns_SRN8040TA
Connections:
- net 12V: now also C2.1
- net GND: now also C2.2
Other:
- moved on the sheet: C1
Changed lines of the file:
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@@
+	)
+	(junction
+		(at 33.02 86.36)
+		(diameter 0)
+		(color 0 0 0 0)
 	)
 	(junction
@@
 	)
 	(junction
-		(at 35.56 86.36)
+		(at 48.26 86.36)
 		(diameter 0)
 		(color 0 0 0 0)
@@
 	(wire
 		(pts
+			(xy 33.02 86.36) (xy 48.26 86.36)
+		)
+		(stroke
+			(width 0)
+			(type default)
+		)
+	)
+	(wire
+		(pts
 			(xy 143.51 86.36) (xy 143.51 119.38)
 		)
@@
 	(wire
 		(pts
+			(xy 48.26 86.36) (xy 87.63 86.36)
+		)
+		(stroke
+			(width 0)
+			(type default)
+		)
+	)
+	(wire
+		(pts
 			(xy 99.06 64.77) (xy 137.16 64.77)
 		)
@@
 	(wire
 		(pts
+			(xy 33.02 121.92) (xy 33.02 139.7)
+		)
+		(stroke
+			(width 0)
+			(type default)
+		)
+	)
+	(wire
+		(pts
+			(xy 48.26 86.36) (xy 48.26 114.3)
+		)
+		(stroke
+			(width 0)
+			(type default)
+		)
+	)
+	(wire
+		(pts
 			(xy 111.76 52.07) (xy 111.76 44.45)
 		)
@@
 	(wire
 		(pts
+			(xy 48.26 121.92) (xy 48.26 139.7)
+		)
+		(stroke
+			(width 0)
+			(type default)
+		)
+	)
+	(wire
+		(pts
 			(xy 151.13 100.33) (xy 158.75 100.33)
 		)
@@
 	(wire
 		(pts
-			(xy 25.4 86.36) (xy 35.56 86.36)
+			(xy 25.4 86.36) (xy 33.02 86.36)
 		)
 		(stroke
@@
 	(wire
 		(pts
-			(xy 35.56 121.92) (xy 35.56 139.7)
-		)
-		(stroke
-			(width 0)
-			(type default)
-		)
-	)
-	(wire
-		(pts
 			(xy 158.75 100.33) (xy 158.75 102.87)
 		)
@@
 	(wire
 		(pts
-			(xy 35.56 86.36) (xy 87.63 86.36)
-		)
-		(stroke
-			(width 0)
-			(type default)
-		)
-	)
-	(wire
-		(pts
 			(xy 124.46 86.36) (xy 124.46 96.52)
 		)
@@
 	(wire
 		(pts
-			(xy 35.56 114.3) (xy 35.56 86.36)
+			(xy 33.02 114.3) (xy 33.02 86.36)
 		)
 		(stroke
@@
 		)
 	)
+	(hierarchical_label "GND"
+		(shape input)
+		(at 48.26 139.7 270)
+		(effects
+			(font
+				(size 1.27 1.27)
+			)
+			(justify right)
+		)
+	)
 	(hierarchical_label "3.3V"
 		(shape output)
@@
 	(hierarchical_label "GND"
 		(shape input)
-		(at 35.56 139.7 270)
+		(at 33.02 139.7 270)
 		(effects
 			(font
@@
 			)
 		)
-		(property "Footprint" "Inductor_SMD:L_1210_3225Metric"
+		(property "Footprint" "Inductor_SMD:L_Bourns_SRN8040TA"
 			(at 127 44.45 0)
 			(effects
@@
 	)
 	(symbol
+		(lib_id "Device:C")
+		(at 48.26 118.11 0)
+		(unit 1)
+		(exclude_from_sim no)
+		(in_bom yes)
+		(on_board yes)
+		(dnp no)
+		(property "Reference" "C2"
+			(at 52.07 116.8399 0)
+			(effects
+				(font
+					(size 1.27 1.27)
+				)
+				(justify left)
+			)
+		)
+		(property "Value" "100nF"
+			(at 52.07 119.126 0)
+			(effects
+				(font
+					(size 1.27 1.27)
+				)
+				(justify left)
+			)
+		)
+		(property "Footprint" "Capacitor_SMD:C_0805_2012Metric"
+			(at 49.2252 121.92 0)
+			(effects
+				(font
+					(size 1.27 1.27)
+				)
+				(hide yes)
+			)
+		)
+		(property "Datasheet" "~"
+			(at 48.26 118.11 0)
+			(effects
+				(font
+					(size 1.27 1.27)
+				)
+				(hide yes)
+			)
+		)
+		(property "Description" "Unpolarized capacitor"
+			(at 48.26 118.11 0)
+			(effects
+				(font
+					(size 1.27 1.27)
+				)
+				(hide yes)
+			)
+		)
+		(pin "1"
+		)
+		(pin "2"
+		)
+		(instances
+			(project "nixie_clock"
+				(path "/90430e5f-7049-4de8-b92d-f897c4a89819/3e544bdc-8ef6-4ae7-86a5-8f5d44c9c569"
+					(reference "C2")
+					(unit 1)
+				)
+			)
+		)
+	)
+	(symbol
 		(lib_id "Regulator_Switching:MAX1771xSA")
 		(at 87.63 106.68 0)
@@
 	(symbol
 		(lib_id "Device:C_Polarized")
-		(at 35.56 118.11 0)
+		(at 33.02 118.11 0)
 		(unit 1)
 		(exclude_from_sim no)
@@
 		(fields_autoplaced yes)
 		(property "Reference" "C1"
-			(at 39.37 115.9509 0)
+			(at 36.83 115.9509 0)
 			(effects
 				(font
@@
 		)
 		(property "Value" "100uF"
-			(at 39.37 118.4909 0)
+			(at 36.83 118.4909 0)
 			(effects
 				(font
@@
 		)
 		(property "Footprint" "Capacitor_Tantalum_SMD:CP_EIA-7343-31_Kemet-D_HandSolder"
-			(at 36.5252 121.92 0)
+			(at 33.9852 121.92 0)
 			(effects
 				(font
@@
 		)
 		(property "Datasheet" "~"
-			(at 35.56 118.11 0)
+			(at 33.02 118.11 0)
 			(effects
 				(font
@@
 		)
 		(property "Description" "Polarized capacitor"
-			(at 35.56 118.11 0)
-			(effects
-				(font
+			(at 33.02 118.11 0)
+			(effects
+				(font
