File: hardware/power_supply.kicad_sch (KiCad schematic)
At the start: 23 parts, among them Q1 IRF740, U1 AP63203WU, U2 MAX1771xSA

Commit message: Add 3314J potentiometer. Found L2 LCSC part number.
Parts:
- RV1: footprint Potentiometer_SMD:Potentiometer_Bourns_3224G_Horizontal -> Potentiometer_SMD:Potentiometer_Bourns_3314J_Vertical
Changed lines of the file:
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@@
 			)
 		)
-		(property "Footprint" "Potentiometer_SMD:Potentiometer_Bourns_3224G_Horizontal"
+		(property "Footprint" "Potentiometer_SMD:Potentiometer_Bourns_3314J_Vertical"
 			(at 158.75 106.68 0)
 			(effects
